Commit message: Update (Unsaved).xacro

File: task/(Unsaved)_description/urdf/(Unsaved).xacro (robot description, xacro)
@@ -68,5 +68,5 @@
   <parent link="base_link"/>
   <child link="Component3_1"/>
-  <axis xyz="-0.0 -1.0 0.0"/>
+  <axis xyz="0.0 1.0 0.0"/>
 </joint>
 <joint name="Rev2" type="continuous">
